Commit message: IMU Hardware Interface 初版

File: src/dart_flysystem_hardware/description/control/dart_hardware_ros2_control.urdf.xacro (robot description, xacro)
@@ -51,3 +51,26 @@
         </ros2_control>
     </xacro:macro>
+    <xacro:macro name="dart_sensors_ros2_control" params="name prefix">
+        <!-- IMU and wind wing sensor -->
+        <ros2_control name="${name}" type="sensor">
+            <hardware>
+                <plugin>dart_flysystem_hardware/DartFlySystemHardwareIMU</plugin>
+                <param name="serial_file">/dev/ttyS1</param>
+                <param name="baudrate">230400</param>
+                <param name="imu_address">80</param>
+            </hardware>
+            <sensor name="${prefix}imu">
+                <state_interface name="linear_acceleration.x" />
+                <state_interface name="linear_acceleration.y" />
+                <state_interface name="linear_acceleration.z" />
+                <state_interface name="angular_velocity.x" />
+                <state_interface name="angular_velocity.y" />
+                <state_interface name="angular_velocity.z" />
+                <state_interface name="orientation.x" />
+                <state_interface name="orientation.y" />
+                <state_interface name="orientation.z" />
+                <state_interface name="orientation.w" />
+            </sensor>
+        </ros2_control>
+    </xacro:macro>
 </robot>

File: src/dart_flysystem_hardware/description/urdf/dart_hardware_test.urdf.xacro (robot description, xacro)
@@ -7,3 +7,4 @@
     <xacro:dart prefix="dart_" parent="base_link"/>
     <xacro:dart_servo_ros2_control name="DartServo" prefix="dart_" />
+    <xacro:dart_sensors_ros2_control name="DartSensors" prefix="dart_" />
 </robot>

Commit message: 完成I2C-磁编码器/电机油门控制/MCU完成部分PID调节

File: src/dart_flysystem_hardware/description/control/dart_hardware_ros2_control.urdf.xacro (robot description, xacro)
@@ -5,5 +5,5 @@
         <ros2_control name="${name}" type="system">
             <hardware>
-                <plugin>dart_flysystem_hardware/DartFlySystemHardwareServo</plugin>
+                <plugin>dart_flysystem_hardware/DartFlySystemHardwareActuator</plugin>
                 <param name="debug">true</param>
                 <param name="offset_angle">${PI/2}</param>
@@ -49,7 +49,36 @@
                 <param name="pwm_channel"> 0</param>
             </joint>
+            <joint name="${prefix}base_link_to_throttle_joint">
+                <command_interface name="velocity">
+                </command_interface>
+                <state_interface name="velocity" />
+                <!-- pwm9@fe6f0010 -->
+                <param name="pwm_chip">1</param>
+                <param name="pwm_channel"> 0</param>
+                <param name="default_velocity">0.1</param>
+                <param name="max_velocity_duty_cycle_percentage">80</param>
+                <param name="min_velocity_duty_cycle_percentage">62</param>
+                <param name="pwm_frequency">500</param>
+            </joint>
         </ros2_control>
     </xacro:macro>
-    <xacro:macro name="dart_sensors_ros2_control" params="name prefix">
+    <xacro:macro name="dart_encoder_ros2_control" params="name prefix">
+        <!-- Wind wing sensor -->
+        <ros2_control name="${name}" type="sensor">
+            <hardware>
+                <plugin>dart_flysystem_hardware/DartFlySystemHardwareEncoder</plugin>
+                <param name="i2c_device">/dev/i2c-4</param>
+                <param name="i2c_address">0x36</param>
+                <param name="encoder_raw_offset">0</param>
+                <!-- encoder_offset直接作用于原始角度值，单位是4096/rad -->
+                <param name="dart_i2c_en_path">/sys/class/leds/dart-i2c-en/brightness</param>
+            </hardware>
+            <sensor name="${prefix}encoder">
+                <state_interface name="position" />
+                <state_interface name="velocity" />
+            </sensor>
+        </ros2_control>
+    </xacro:macro>
+    <xacro:macro name="dart_imu_ros2_control" params="name prefix">
         <!-- IMU and wind wing sensor -->
         <ros2_control name="${name}" type="sensor">
